Commit message: update

File: src/robot_arm_moveit/config/.ipynb_checkpoints/temp-checkpoint.urdf (robot description, URDF)
Before this commit: robot robot_arm, 9 links, 8 joints
Links:
- removed link link_7_1
- removed link link_8_1
- link base_link: mass None -> 2.200366644976027; geometry collision mesh filename=package://robot_arm_description/meshes/base_link.stl scale=0.001 0.001 0.001; visual mesh filename=package://robot_arm_description/meshes/base_link.stl scale=0.001 0.001 0.001
Joints:
- removed joint joint_7
- removed joint joint_8
- joint joint_1: limit (none) -> lower=-2.443461 upper=2.443461 effort=100 velocity=100
- joint joint_2: limit lower=-0.872665 upper=1.570796 effort=100 velocity=100 -> lower=-1.570796 upper=1.570796 effort=100 velocity=100
- joint joint_4: limit (none) -> lower=-2.443461 upper=2.443461 effort=100 velocity=100
- joint joint_6: limit (none) -> lower=-2.443461 upper=2.443461 effort=100 velocity=100

File: src/robot_arm_moveit/config/temp.urdf (robot description, URDF)
Before this commit: robot robot_arm, 7 links, 6 joints
Joints:
- joint joint_1: limit (none) -> lower=-2.443461 upper=2.443461 effort=100 velocity=100
- joint joint_2: limit lower=-0.872665 upper=1.570796 effort=100 velocity=100 -> lower=-1.570796 upper=1.570796 effort=100 velocity=100
- joint joint_4: limit (none) -> lower=-2.443461 upper=2.443461 effort=100 velocity=100
- joint joint_6: limit (none) -> lower=-2.443461 upper=2.443461 effort=100 velocity=100
