Commit message: test

File: src/three/urdf/gazebo_robot_arm.urdf (robot description, URDF)
Before this commit: robot urdf_assembly_2, 8 links, 7 joints
Joints:
- joint joint_7: axis (none) -> 1.0 0.0 0.0; limit (none) -> lower=-3.141593 upper=3.141593 effort=100 velocity=100; type fixed -> revolute
